Commit message: feat: add a robot description node

File: mujoco_ros2_base/sample_xml/pendulum.urdf (robot description, URDF)
Before this commit: robot pendulum, 3 links, 2 joints
Links:
- link world: mass 0.0 -> None

Commit message: fix: correct urdf visuals

File: mujoco_ros2_base/sample_xml/pendulum.urdf (robot description, URDF)
Before this commit: robot pendulum, 3 links, 2 joints
Links:
- removed link hinge_jointbody
- removed link world
- added link base; visual cylinder length=0.06 radius=0.021
- added link mass, mass 1.0; visual sphere radius=0.05
- link pole: mass 1.0 -> 0.001; geometry visual cylinder length=0.5 radius=0.02
Joints:
- removed joint hinge_offset
- added joint glue: type fixed, parent pole, child mass, origin xyz=-0.0 -0.0 -0.0 rpy=0.0 0.0 0.0
- joint hinge: axis 0.0 1.0 0.0 -> 1.0 0.0 0.0; child hinge_jointbody -> pole; origin xyz=0.0 0.0 0.6 rpy=0.0 0.0 0.0 -> xyz=0.0 0.0 0.25 rpy=0.0 0.0 0.0; parent world -> base

Commit message: fix: fix visuals

File: mujoco_ros2_base/sample_xml/pendulum.urdf (robot description, URDF)
Before this commit: robot pendulum, 3 links, 2 joints
Joints:
- joint hinge: origin xyz=0.0 0.0 0.25 rpy=0.0 0.0 0.0 -> xyz=0.0 0.0 0.0 rpy=0.0 0.0 0.0
